File: pcb/handheld/audio.kicad_sch (KiCad schematic)
At the start: 23 parts, among them J1401 Headphone Jack, J1402 Speaker_Left/Mono, J1403 Speaker_Right, Q3 AO3400A, U1401 TLV320DAC3101

Commit message: Rev A of PCB
Parts:
- added J601: TP_I2S, Connector_PinSocket_2.54mm:PinSocket_1x04_P2.54mm_Vertical, symbol Connector_Generic:Conn_01x04
- J1601: renamed from J1402; value Speaker_Left/Mono -> SPK_L
- J1602: renamed from J1403; value Speaker_Right -> SPK_R
- renumbered C1407 to C1601, C1409 to C1603, C18 to C1605, C18 to C1607, C1411 to C1609, C1413 to C1611, C1402 to C1613, C1403 to C1614, J1401 to J1603, R10 to R1602, R1404 to R1603, R11 to R1604, U1401 to U1601
Connections:
- net DAC_BCLK: now also J601.2 (Pin_2)
- net DAC_DIN: now also J601.4 (Pin_4)
- net DAC_MCLK: now also J601.1 (Pin_1)
- net DAC_WCLK: now also J601.3 (Pin_3)
- net GND: now also J1603.R2
- net MICBIAS: now reaches R1603.1, U1601.12 (MICBIAS)
- net +1V8_DAC renamed +1V8
- net +3V3_DAC renamed +3V3_FPGA
- net RP2040_~{IRQ} renamed MCU_~{IRQ}
Other:
- note added: "Test Points"
- note added: "nFET converts push-pull active-high DAC interrupt into open-drain active-low MCU_~{INT}"
- note removed: "nFET converts push-pull active-high DAC interrupt into open-drain active-low RP2040_~{INT}"
