File: pcb/handheld/buttons.kicad_sch (KiCad schematic)
At the start: 46 parts, among them SW1601 SW_Push, SW1602 BTN_A, SW1603 BTN_Home, SW1604 BTN_Select, SW1605 BTN_Start, SW1606 BTN_Y, SW1607 BTN_B, SW1608 BTN_X, SW1609 BTN_LEFT, SW1610 BTN_UP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

Commit message: Rev A of PCB
Parts:
- removed SW1601: SW_Push, symbol Switch:SW_Push
- added C1: 100n, Capacitor_SMD:C_0402_1005Metric, symbol Device:C_Small
- added U1501: TCA9535PWR, Package_SO:TSSOP-24_4.4x7.8mm_P0.65mm, symbol Interface_Expansion:TCA9535PWR
- SW1501: renamed from SW1610; value BTN_UP -> Up; footprint (none) -> Game_Bub:SW_SPST_SKRR; LCSC (none) -> C97437
- SW1502: renamed from SW1613; value BTN_L -> L; footprint (none) -> Game_Bub:SW_Tactile_SPST_Angled_TL1105VFxxxx
- SW1503: renamed from SW1614; value BTN_R -> R; footprint (none) -> Game_Bub:SW_Tactile_SPST_Angled_TL1105VFxxxx
- SW1504: renamed from SW1608; value BTN_X -> X; footprint (none) -> Game_Bub:SW_SPST_SKRR; LCSC (none) -> C97437
- SW1505: renamed from SW1609; value BTN_LEFT -> Left; footprint (none) -> Game_Bub:SW_SPST_SKRR; LCSC (none) -> C97437
- SW1506: renamed from SW1612; value BTN_RIGHT -> Right; footprint (none) -> Game_Bub:SW_SPST_SKRR; LCSC (none) -> C97437
- SW1507: renamed from SW1606; value BTN_Y -> Y; footprint (none) -> Game_Bub:SW_SPST_SKRR; LCSC (none) -> C97437
- SW1508: renamed from SW1602; value BTN_A -> A; footprint (none) -> Game_Bub:SW_SPST_SKRR; LCSC (none) -> C97437
- SW1509: renamed from SW1611; value BTN_DOWN -> Down; footprint (none) -> Game_Bub:SW_SPST_SKRR; LCSC (none) -> C97437
- SW1510: renamed from SW1607; value BTN_B -> B; footprint (none) -> Game_Bub:SW_SPST_SKRR; LCSC (none) -> C97437
- SW1511: renamed from SW1604; value BTN_Select -> Select; footprint (none) -> Game_Bub:SW_SPST_SKRB; LCSC (none) -> C115356
- SW1512: renamed from SW1603; value BTN_Home -> Home; footprint (none) -> Game_Bub:SW_SPST_SKRB; LCSC (none) -> C115356
- SW1513: renamed from SW1605; value BTN_Start -> Start; footprint (none) -> Game_Bub:SW_SPST_SKRB; LCSC (none) -> C115356
- SW1514: renamed from SW1616; value BTN_Vol_Up -> Vol_Up; footprint (none) -> Game_Bub:SW_SPST_SKSC; LCSC (none) -> C115361
- SW1515: renamed from SW1615; value BTN_Vol_Down -> Vol_Down; footprint (none) -> Game_Bub:SW_SPST_SKSC; LCSC (none) -> C115361
- renumbered R11 to R31
Connections:
- net +3V3: now also C1.1, U1501.24 (VCC)
- net BTN_A: now also U1501.7 (P03)
- net BTN_B: now also U1501.8 (P04)
- net BTN_L: now also U1501.14 (P11)
- net BTN_R: now also U1501.4 (P00)
- net BTN_X: now also U1501.5 (P01)
- net BTN_Y: now also U1501.6 (P02)
- net GND: now also C1.2, U1501.10 (P06), U1501.11 (P07), U1501.12 (GND), U1501.13 (P10), U1501.2 (A1), U1501.21 (A0), U1501.3 (A2)
- net BTN_B_s: now reaches R31.2, R31.2, SW1510.1
- net BTN_Home_s: now reaches R31.2, R31.2, SW1512.1
- net BTN_Up_s: now reaches R31.2, R31.2, SW1501.1
- net BTN_Left_s: now reaches R31.2, R31.2, SW1505.1
- net BTN_Down_s: now reaches R31.2, R31.2, SW1509.1
- net BTN_Vol_Down_s: now reaches R31.2, R31.2, SW1515.1
- net BTN_Select_s: now reaches R31.2, R31.2, SW1511.1
- net BTN_Start_s: now reaches R31.2, R31.2, SW1513.1
- net BTN_Y_s: now reaches R31.2, R31.2, SW1507.1
- net BTN_Vol_Up_s: now reaches R31.2, R31.2, SW1514.1
- net BTN_L_s: now reaches R31.2, R31.2, SW1502.1
- net BTN_Right_s: now reaches R31.2, R31.2, SW1506.1
- net BTN_A_s: now reaches R31.2, R31.2, SW1508.1
- net BTN_X_s: now reaches R31.2, R31.2, SW1504.1
- net BTN_R_s: now reaches R31.2, R31.2, SW1503.1
- net BTN_DOWN renamed BTN_Down
- net BTN_Down: now also U1501.18 (P15)
- net BTN_HOME renamed BTN_Home
- net BTN_LEFT renamed BTN_Left
- net BTN_Left: now also U1501.17 (P14)
- net BTN_RIGHT renamed BTN_Right
- net BTN_Right: now also U1501.16 (P13)
- net BTN_SELECT renamed BTN_Select
- net BTN_Select: now also U1501.19 (P16)
- net BTN_START renamed BTN_Start
- net BTN_Start: now also U1501.20 (P17)
- net BTN_UP renamed BTN_Up
- net BTN_Up: now also U1501.15 (P12)
- new net HDMI_~{HPD}: U1501.9 (P05)
- new net I2C0_SCL: U1501.22 (SCL)
- new net I2C0_SDA: U1501.23 (SDA)
- new net MCU_~{IRQ}: U1501.1 (~{INT})
Other:
- note added: "Button I/O Expander (optional)"
- note added: "I2C Addr: 0x20"
- moved on the sheet: R31, SW1501, SW1502, SW1503, SW1504, SW1505, SW1506, SW1507, SW1508, SW1509, SW1510, SW1511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
