File: pcb/handheld/fpga_io_14.kicad_sch (KiCad schematic)
At the start: 8 parts, among them J601 FPGA_JTAG, U501 XC7A100T-CSG324, X601 YSO110TR 50MHz

Commit message: Rev A of PCB
Parts:
- removed C1: 100n, Capacitor_SMD:C_0402_1005Metric, symbol Device:C_Small
- removed C58: 47u, Capacitor_SMD:C_0805_2012Metric, symbol Device:C_Small
- removed J601: FPGA_JTAG, Connector_PinSocket_2.54mm:PinSocket_1x04_P2.54mm_Vertical, symbol Connector_Generic:Conn_01x04
- removed R601, R602, R603: 4K7, Resistor_SMD:R_0402_1005Metric, symbol Device:R_Small
- removed U501: XC7A100T-CSG324, Package_BGA:Xilinx_CSG324, symbol Game_Bub:XC7A100T-CSG324
- removed X601: YSO110TR 50MHz, Oscillator:Oscillator_SMD_SeikoEpson_SG8002CE-4Pin_3.2x2.5mm, symbol Game_Bub:YSO110TR
- added C626, C627: 4u7, Capacitor_SMD:C_0402_1005Metric, symbol Device:C_Small
- added C628, C629, C630, C631: 470n, Capacitor_SMD:C_0402_1005Metric, symbol Device:C_Small
- added D102: H5VU25U, Package_DFN_QFN:Diodes_UDFN-10_1.0x2.5mm_P0.5mm, symbol Game_Bub:H5VU25U
- added J802: PMOD, Game_Bub:PinSocket_1x06_P2.54mm_Horizontal_SMD, symbol Connector_Generic:Conn_01x06
- added R701: 1K, Resistor_SMD:R_0402_1005Metric, symbol Device:R_Small
- added U501: XC7A100T-CSG324, Package_BGA:Xilinx_CSG324, symbol Game_Bub:XC7A100T-CSG324
Connections:
- net +3V3_FPGA: now also C626.1, C627.1, C628.1, C629.1, C630.1, C631.1, J802.1 (Pin_1), R701.2, U501.L17 (VCCO_14), U501.N13 (VCCO_14), U501.P16 (VCCO_14), U501.T12 (VCCO_14), U501.U15 (VCCO_14), U501.V18 (VCCO_14)
- net GND: now also C626.2, C627.2, C628.2, C629.2, C630.2, C631.2, D102.3 (A), D102.8 (A), J802.2 (Pin_2)
- new net FPGA_PUDC_B: R701.1, U501.L15 (IO_L3P_T0_DQS_PUDC_B_14)
- new net GB_Dir_SO: U501.L14 (IO_L2P_T0_D02_14)
- new net GB_Link_SO: U501.L13 (IO_L6P_T0_FCS_B_14)
- new net LCD_DB10: U501.L18 (IO_L4P_T0_D04_14)
- new net LCD_DB11: U501.K17 (IO_L1P_T0_D00_MOSI_14)
- new net PMOD_1: D102.5 (K4), D102.6 (K4), J802.6 (Pin_6), U501.M14 (IO_L2N_T0_D03_14)
- new net PMOD_2: D102.4 (K3), D102.7 (K3), J802.5 (Pin_5), U501.N14 (IO_L8P_T1_D11_14)
- new net PMOD_3: D102.2 (K2), D102.9 (K2), J802.4 (Pin_4), U501.P14 (IO_L8N_T1_D12_14)
- new net PMOD_4: D102.1 (K1), D102.10 (K1), J802.3 (Pin_3), U501.M13 (IO_L6N_T0_D08_VREF_14)
- new net SPI2_PICO/D0: U501.K18 (IO_L1N_T0_D01_DIN_14)
- new net SRAM_A0: U501.N17 (IO_L9P_T1_DQS_14)
- new net SRAM_A1: U501.M17 (IO_L10N_T1_D15_14)
- new net SRAM_A10: U501.V12 (IO_L20N_T3_A07_D23_14)
- new net SRAM_A11: U501.U11 (IO_L19N_T3_A09_D25_VREF_14)
- new net SRAM_A12: U501.V11 (IO_L21N_T3_DQS_A06_D22_14)
- new net SRAM_A13: U501.V10 (IO_L21P_T3_DQS_14)
- new net SRAM_A14: U501.U12 (IO_L20P_T3_A08_D24_14)
- new net SRAM_A15: U501.R18 (IO_L7P_T1_D09_14)
- new net SRAM_A16: U501.P17 (IO_L12P_T1_MRCC_14)
- new net SRAM_A17: U501.P18 (IO_L9N_T1_DQS_D13_14)
- new net SRAM_A2: U501.M18 (IO_L4N_T0_D05_14)
- new net SRAM_A3: U501.T9 (IO_L24P_T3_A01_D17_14)
- new net SRAM_A4: U501.T10 (IO_L24N_T3_A00_D16_14)
- new net SRAM_A5: U501.P15 (IO_L13P_T2_MRCC_14)
- new net SRAM_A6: U501.N16 (IO_L11N_T1_SRCC_14)
- new net SRAM_A7: U501.N15 (IO_L11P_T1_SRCC_14)
- new net SRAM_A8: U501.M16 (IO_L10P_T1_D14_14)
- new net SRAM_A9: U501.L16 (IO_L3N_T0_DQS_EMCCLK_14)
- new net SRAM_IO0: U501.R11 (IO_0_14)
- new net SRAM_IO1: U501.R12 (IO_L5P_T0_D06_14)
- new net SRAM_IO10: U501.U14 (IO_L22P_T3_A05_D21_14)
- new net SRAM_IO11: U501.V15 (IO_L16P_T2_CSI_B_14)
- new net SRAM_IO12: U501.V16 (IO_L16N_T2_A15_D31_14)
- new net SRAM_IO13: U501.U16 (IO_L18P_T2_A12_D28_14)
- new net SRAM_IO14: U501.V17 (IO_L18N_T2_A11_D27_14)
- new net SRAM_IO15: U501.U18 (IO_L17N_T2_A13_D29_14)
- new net SRAM_IO2: U501.T13 (IO_L23P_T3_A03_D19_14)
- new net SRAM_IO3: U501.R13 (IO_L5N_T0_D07_14)
- new net SRAM_IO4: U501.T14 (IO_L14P_T2_SRCC_14)
- new net SRAM_IO5: U501.T15 (IO_L14N_T2_SRCC_14)
- new net SRAM_IO6: U501.T16 (IO_L15N_T2_DQS_DOUT_CSO_B_14)
- new net SRAM_IO7: U501.R16 (IO_L15P_T2_DQS_RDWR_B_14)
- new net SRAM_IO8: U501.U13 (IO_L23N_T3_A02_D18_14)
- new net SRAM_IO9: U501.V14 (IO_L22N_T3_A04_D20_14)
- new net SRAM_~{CE}: U501.R10 (IO_25_14)
- new net SRAM_~{LB}: U501.U17 (IO_L17P_T2_A14_D30_14)
- new net SRAM_~{OE}: U501.R17 (IO_L12N_T1_MRCC_14)
- new net SRAM_~{UB}: U501.T18 (IO_L7N_T1_D10_14)
- new net SRAM_~{WE}: U501.R15 (IO_L13N_T2_MRCC_14)
- no-connect marks 0 -> 1
Other:
- note added: "PMOD"
- note added: "PUDC_B high disables pull-ups during boot"
- note removed: "ADC unused"
- note removed: "CFGBVS = 1 for 3.3V config"
- note removed: "Clock Source 50 MHz"
- note removed: "Configuration Modes M[2:0]"
- note removed: "JTAG 101 Slave Serial 111"
- note removed: "Temperature-sensing diode not used"
- note removed: "V_{CCO} Bank 0: 1x 47 µF"
