File: pcb/handheld/fpga_io_15.kicad_sch (KiCad schematic)
At the start: 30 parts, among them U501 XC7A100T-CSG324

Commit message: Rev A of PCB
Parts:
- removed C33 (x5): 100u, Capacitor_SMD:C_1206_3216Metric, symbol Device:C_Small
- removed C505, C506, C507, C508, C509, C510, C523, C524: 4u7, Capacitor_SMD:C_0402_1005Metric, symbol Device:C_Small
- removed C511, C512, C513, C514, C515, C516, C517, C518, C520, C521, C525, C526, C527, C528: 470n, Capacitor_SMD:C_0402_1005Metric, symbol Device:C_Small
- removed C522, C529: 47u, Capacitor_SMD:C_0805_2012Metric, symbol Device:C_Small
- removed U501: XC7A100T-CSG324, Package_BGA:Xilinx_CSG324, symbol Game_Bub:XC7A100T-CSG324
- added C626, C627: 4u7, Capacitor_SMD:C_0402_1005Metric, symbol Device:C_Small
- added C628, C629, C630, C631: 470n, Capacitor_SMD:C_0402_1005Metric, symbol Device:C_Small
- added U501: XC7A100T-CSG324, Package_BGA:Xilinx_CSG324, symbol Game_Bub:XC7A100T-CSG324
Connections:
- net +3V3_FPGA: now also C626.1, C627.1, C628.1, C629.1, C630.1, C631.1, U501.A17 (VCCO_15), U501.C13 (VCCO_15), U501.D16 (VCCO_15), U501.G15 (VCCO_15), U501.H18 (VCCO_15), U501.K14 (VCCO_15)
- net GND: now also C626.2, C627.2, C628.2, C629.2, C630.2, C631.2
- new net GB_3V3_Enable: U501.B16 (IO_L7P_T1_AD2P_15)
- new net GB_5V_Enable: U501.J13 (IO_L17N_T2_A25_15)
- new net GB_Cart_A16: U501.A11 (IO_L4N_T0_15)
- new net GB_Cart_A17: U501.B12 (IO_L3N_T0_DQS_AD1N_15)
- new net GB_Cart_A18: U501.A13 (IO_L9P_T1_DQS_AD3P_15)
- new net GB_Cart_A19: U501.B13 (IO_L2P_T0_AD8P_15)
- new net GB_Cart_A20: U501.A14 (IO_L9N_T1_DQS_AD3N_15)
- new net GB_Cart_A21: U501.B14 (IO_L2N_T0_AD8N_15)
- new net GB_Cart_A22: U501.A15 (IO_L8P_T1_AD10P_15)
- new net GB_Cart_A23: U501.B11 (IO_L4P_T0_15)
- new net GB_Cart_AD10: U501.D12 (IO_L6P_T0_15)
- new net GB_Cart_AD11: U501.D13 (IO_L6N_T0_VREF_15)
- new net GB_Cart_AD12: U501.C14 (IO_L1N_T0_AD0N_15)
- new net GB_Cart_AD13: U501.D14 (IO_L1P_T0_AD0P_15)
- new net GB_Cart_AD14: U501.C15 (IO_L12N_T1_MRCC_15)
- new net GB_Cart_AD15: U501.C16 (IO_L20P_T3_A20_15)
- new net GB_Cart_AD9: U501.C12 (IO_L3P_T0_DQS_AD1P_15)
- new net GB_Cart_VIN: U501.C17 (IO_L20N_T3_A19_15)
- new net GB_Cart_~{CS2}: U501.B17 (IO_L7N_T1_AD2N_15)
- new net GB_Dir_Cart0: U501.A16 (IO_L8N_T1_AD10N_15)
- new net GB_Dir_SC: U501.G14 (IO_L15N_T2_DQS_ADV_B_15)
- new net GB_Dir_SD: U501.F13 (IO_L5P_T0_AD9P_15)
- new net GB_Dir_SI: U501.H14 (IO_L15P_T2_DQS_15)
- new net GB_Dir_VIN: U501.B18 (IO_L10P_T1_AD11P_15)
- new net GB_Dir_~{CS2}: U501.A18 (IO_L10N_T1_AD11N_15)
- new net GB_Link_SC: U501.G13 (IO_0_15)
- new net GB_Link_SD: U501.F14 (IO_L5N_T0_AD9N_15)
- new net GB_Link_SI: U501.J14 (IO_L19P_T3_A22_15)
- new net LCD_DATA_EN: U501.F18 (IO_L22N_T3_A16_15)
- new net LCD_DB0: U501.K16 (IO_25_15)
- new net LCD_DB1: U501.K15 (IO_L24P_T3_RS1_15)
- new net LCD_DB12: U501.J17 (IO_L23P_T3_FOE_B_15)
- new net LCD_DB13: U501.J18 (IO_L23N_T3_FWE_B_15)
- new net LCD_DB14: U501.H17 (IO_L18P_T2_A24_15)
- new net LCD_DB15: U501.H16 (IO_L13P_T2_MRCC_15)
- new net LCD_DB16: U501.G18 (IO_L22P_T3_A17_15)
- new net LCD_DB17: U501.G17 (IO_L18N_T2_A23_15)
- new net LCD_DB2: U501.J15 (IO_L24N_T3_RS0_15)
- new net LCD_DB3: U501.H15 (IO_L19N_T3_A21_VREF_15)
- new net LCD_DB4: U501.G16 (IO_L13N_T2_MRCC_15)
- new net LCD_DB5: U501.F16 (IO_L14N_T2_SRCC_15)
- new net LCD_DB6: U501.F15 (IO_L14P_T2_SRCC_15)
- new net LCD_DB7: U501.E16 (IO_L11N_T1_SRCC_15)
- new net LCD_DB8: U501.E15 (IO_L11P_T1_SRCC_15)
- new net LCD_DB9: U501.D15 (IO_L12P_T1_MRCC_15)
- new net LCD_DOTCLK: U501.E17 (IO_L16P_T2_A28_15)
- new net LCD_HSYNC: U501.E18 (IO_L21P_T3_DQS_15)
- new net LCD_VSYNC: U501.D17 (IO_L16N_T2_A27_15)
- new net SW_Cartridge: U501.D18 (IO_L21N_T3_DQS_A18_15)
- no-connect marks 0 -> 1
Other:
- note removed: "Bulk decoupling capacitor shared between 4x IO banks sharing same VCCO (3.3V)"
