File: pcb/handheld/fpga_io_16.kicad_sch (KiCad schematic)
At the start: 30 parts, among them U501 XC7A100T-CSG324

Commit message: Rev A of PCB
Parts:
- removed C33 (x5): 100u, Capacitor_SMD:C_1206_3216Metric, symbol Device:C_Small
- removed C505, C506, C507, C508, C509, C510, C523, C524: 4u7, Capacitor_SMD:C_0402_1005Metric, symbol Device:C_Small
- removed C511, C512, C513, C514, C515, C516, C517, C518, C520, C521, C525, C526, C527, C528: 470n, Capacitor_SMD:C_0402_1005Metric, symbol Device:C_Small
- removed C522, C529: 47u, Capacitor_SMD:C_0805_2012Metric, symbol Device:C_Small
- removed U501: XC7A100T-CSG324, Package_BGA:Xilinx_CSG324, symbol Game_Bub:XC7A100T-CSG324
- added U501: XC7A100T-CSG324, Package_BGA:Xilinx_CSG324, symbol Game_Bub:XC7A100T-CSG324
Connections:
- new net BANK16_VCCO: U501.A10 (IO_L14P_T2_SRCC_16), U501.A8 (IO_L12N_T1_MRCC_16), U501.A9 (IO_L14N_T2_SRCC_16), U501.B10 (VCCO_16), U501.B8 (IO_L12P_T1_MRCC_16), U501.B9 (IO_L11N_T1_SRCC_16), U501.C10 (IO_L13N_T2_MRCC_16), U501.C11 (IO_L13P_T2_MRCC_16), U501.C9 (IO_L11P_T1_SRCC_16), U501.D10 (IO_L19N_T3_VREF_16), U501.D9 (IO_L6N_T0_VREF_16)
Other:
- note removed: "Bulk decoupling capacitor shared between 4x IO banks sharing same VCCO (3.3V)"
