File: pcb/handheld/fpga_io_34.kicad_sch (KiCad schematic)
At the start: 30 parts, among them U501 XC7A100T-CSG324

Commit message: Rev A of PCB
Parts:
- removed C33 (x5): 100u, Capacitor_SMD:C_1206_3216Metric, symbol Device:C_Small
- removed C505, C506, C507, C508, C509, C510, C523, C524: 4u7, Capacitor_SMD:C_0402_1005Metric, symbol Device:C_Small
- removed C511, C512, C513, C514, C515, C516, C517, C518, C520, C521, C525, C526, C527, C528: 470n, Capacitor_SMD:C_0402_1005Metric, symbol Device:C_Small
- removed C522, C529: 47u, Capacitor_SMD:C_0805_2012Metric, symbol Device:C_Small
- removed U501: XC7A100T-CSG324, Package_BGA:Xilinx_CSG324, symbol Game_Bub:XC7A100T-CSG324
- added C626, C627: 4u7, Capacitor_SMD:C_0402_1005Metric, symbol Device:C_Small
- added C628, C629, C630, C631: 470n, Capacitor_SMD:C_0402_1005Metric, symbol Device:C_Small
- added U501: XC7A100T-CSG324, Package_BGA:Xilinx_CSG324, symbol Game_Bub:XC7A100T-CSG324
Connections:
- net +3V3_FPGA: now also C626.1, C627.1, C628.1, C629.1, C630.1, C631.1, U501.K4 (VCCO_34), U501.N3 (VCCO_34), U501.P6 (VCCO_34), U501.T2 (VCCO_34), U501.U5 (VCCO_34), U501.V8 (VCCO_34)
- net GND: now also C626.2, C627.2, C628.2, C629.2, C630.2, C631.2
- new net BTN_A: U501.N5 (IO_L13P_T2_MRCC_34)
- new net BTN_B: U501.P5 (IO_L13N_T2_MRCC_34)
- new net BTN_R: U501.L5 (IO_L6N_T0_VREF_34)
- new net BTN_Start: U501.K5 (IO_L5P_T0_34)
- new net BTN_X: U501.L6 (IO_L6P_T0_34)
- new net BTN_Y: U501.M6 (IO_L18P_T2_34)
- new net SDRAM_0_~{CS}: U501.V1 (IO_L7N_T1_34)
- new net SDRAM_A0: U501.R3 (IO_L11P_T1_SRCC_34)
- new net SDRAM_A1: U501.T3 (IO_L11N_T1_SRCC_34)
- new net SDRAM_A10: U501.P4 (IO_L14P_T2_SRCC_34)
- new net SDRAM_A11: U501.V2 (IO_L9N_T1_DQS_34)
- new net SDRAM_A12: U501.U3 (IO_L8N_T1_34)
- new net SDRAM_A2: U501.T4 (IO_L12N_T1_MRCC_34)
- new net SDRAM_A3: U501.R5 (IO_L19N_T3_VREF_34)
- new net SDRAM_A4: U501.R6 (IO_L19P_T3_34)
- new net SDRAM_A5: U501.T6 (IO_L23N_T3_34)
- new net SDRAM_A6: U501.R7 (IO_L23P_T3_34)
- new net SDRAM_A7: U501.R8 (IO_L24P_T3_34)
- new net SDRAM_A8: U501.T8 (IO_L24N_T3_34)
- new net SDRAM_A9: U501.U2 (IO_L9P_T1_DQS_34)
- new net SDRAM_BS0: U501.N4 (IO_L16N_T2_34)
- new net SDRAM_BS1: U501.P3 (IO_L14N_T2_SRCC_34)
- new net SDRAM_CKE: U501.U4 (IO_L8P_T1_34)
- new net SDRAM_CLK: U501.V4 (IO_L10N_T1_34)
- new net SDRAM_DQ0: U501.P2 (IO_L15P_T2_DQS_34)
- new net SDRAM_DQ1: U501.N2 (IO_L3P_T0_DQS_34)
- new net SDRAM_DQ10: U501.V6 (IO_L20N_T3_34)
- new net SDRAM_DQ11: U501.U7 (IO_L22P_T3_34)
- new net SDRAM_DQ12: U501.V7 (IO_L20P_T3_34)
- new net SDRAM_DQ13: U501.U8 (IO_25_34)
- new net SDRAM_DQ14: U501.U9 (IO_L21P_T3_DQS_34)
- new net SDRAM_DQ15: U501.V9 (IO_L21N_T3_DQS_34)
- new net SDRAM_DQ2: U501.N1 (IO_L3N_T0_DQS_34)
- new net SDRAM_DQ3: U501.M2 (IO_L4N_T0_34)
- new net SDRAM_DQ4: U501.M1 (IO_L1N_T0_34)
- new net SDRAM_DQ5: U501.L1 (IO_L1P_T0_34)
- new net SDRAM_DQ6: U501.M3 (IO_L4P_T0_34)
- new net SDRAM_DQ7: U501.M4 (IO_L16P_T2_34)
- new net SDRAM_DQ8: U501.V5 (IO_L10P_T1_34)
- new net SDRAM_DQ9: U501.U6 (IO_L22N_T3_34)
- new net SDRAM_LDQM: U501.R1 (IO_L17P_T2_34)
- new net SDRAM_UDQM: U501.T5 (IO_L12P_T1_MRCC_34)
- new net SDRAM_~{CAS}: U501.T1 (IO_L17N_T2_34)
- new net SDRAM_~{RAS}: U501.U1 (IO_L7P_T1_34)
- new net SDRAM_~{WE}: U501.R2 (IO_L15N_T2_DQS_34)
- no-connect marks 0 -> 5
Other:
- note removed: "Bulk decoupling capacitor shared between 4x IO banks sharing same VCCO (3.3V)"
