File: pcb/handheld/fpga_io_35.kicad_sch (KiCad schematic)
At the start: 30 parts, among them U501 XC7A100T-CSG324

Commit message: Rev A of PCB
Parts:
- removed C33 (x5): 100u, Capacitor_SMD:C_1206_3216Metric, symbol Device:C_Small
- removed C505, C506, C507, C508, C509, C510, C523, C524: 4u7, Capacitor_SMD:C_0402_1005Metric, symbol Device:C_Small
- removed C511, C512, C513, C514, C515, C516, C517, C518, C520, C521, C525, C526, C527, C528: 470n, Capacitor_SMD:C_0402_1005Metric, symbol Device:C_Small
- removed C522, C529: 47u, Capacitor_SMD:C_0805_2012Metric, symbol Device:C_Small
- removed U501: XC7A100T-CSG324, Package_BGA:Xilinx_CSG324, symbol Game_Bub:XC7A100T-CSG324
- added C626, C627: 4u7, Capacitor_SMD:C_0402_1005Metric, symbol Device:C_Small
- added C628, C629, C630, C631: 470n, Capacitor_SMD:C_0402_1005Metric, symbol Device:C_Small
- added U501: XC7A100T-CSG324, Package_BGA:Xilinx_CSG324, symbol Game_Bub:XC7A100T-CSG324
Connections:
- net +3V3_FPGA: now also C626.1, C627.1, C628.1, C629.1, C630.1, C631.1, U501.A7 (VCCO_35), U501.C3 (VCCO_35), U501.D6 (VCCO_35), U501.F2 (VCCO_35), U501.G5 (VCCO_35), U501.J1 (VCCO_35)
- net GND: now also C626.2, C627.2, C628.2, C629.2, C630.2, C631.2
- new net BTN_Down: U501.H5 (IO_L24N_T3_35)
- new net BTN_L: U501.H6 (IO_L24P_T3_35)
- new net BTN_Left: U501.G6 (IO_L19P_T3_35)
- new net BTN_Right: U501.F5 (IO_0_35)
- new net BTN_Select: U501.J5 (IO_25_35)
- new net BTN_Up: U501.E5 (IO_L5N_T0_AD13N_35)
- new net DAC_BCLK: U501.G3 (IO_L20N_T3_35)
- new net DAC_DIN: U501.J4 (IO_L21P_T3_DQS_35)
- new net DAC_MCLK: U501.G4 (IO_L20P_T3_35)
- new net DAC_WCLK: U501.H4 (IO_L21N_T3_DQS_35)
- new net FPGA_CLK_50MHz: U501.E3 (IO_L12P_T1_MRCC_35)
- new net FPGA_SPI_~{CS}: U501.J2 (IO_L22N_T3_35)
- new net GB_Cart_AD0: U501.B6 (IO_L2N_T0_AD12N_35)
- new net GB_Cart_AD1: U501.A6 (IO_L3P_T0_DQS_AD5P_35)
- new net GB_Cart_AD2: U501.B7 (IO_L2P_T0_AD12P_35)
- new net GB_Cart_AD3: U501.C4 (IO_L7P_T1_AD6P_35)
- new net GB_Cart_AD4: U501.D4 (IO_L11N_T1_SRCC_35)
- new net GB_Cart_AD5: U501.C5 (IO_L1N_T0_AD4N_35)
- new net GB_Cart_AD6: U501.D5 (IO_L11P_T1_SRCC_35)
- new net GB_Cart_AD7: U501.C6 (IO_L1P_T0_AD4P_35)
- new net GB_Cart_AD8: U501.D8 (IO_L4P_T0_35)
- new net GB_Cart_PHI: U501.B3 (IO_L10P_T1_AD15P_35)
- new net GB_Cart_~{CS1}: U501.A5 (IO_L3N_T0_DQS_AD5N_35)
- new net GB_Cart_~{OE}: U501.A3 (IO_L8N_T1_AD14N_35)
- new net GB_Cart_~{RD}: U501.B4 (IO_L7N_T1_AD6N_35)
- new net GB_Cart_~{WR}: U501.A4 (IO_L8P_T1_AD14P_35)
- new net GB_Dir_Cart1: U501.D7 (IO_L6N_T0_VREF_35)
- new net GB_Dir_Cart2: U501.C7 (IO_L4N_T0_35)
- new net GB_Dir_Cart3: U501.B2 (IO_L10N_T1_AD15N_35)
- new net HDMI_CEC: U501.F6 (IO_L19N_T3_VREF_35)
- new net HDMI_CLK+: U501.B1 (IO_L9P_T1_DQS_AD7P_35)
- new net HDMI_CLK-: U501.A1 (IO_L9N_T1_DQS_AD7N_35)
- new net HDMI_D0+: U501.C1 (IO_L16N_T2_35)
- new net HDMI_D0-: U501.C2 (IO_L16P_T2_35)
- new net HDMI_D1+: U501.E2 (IO_L14P_T2_SRCC_35)
- new net HDMI_D1-: U501.D2 (IO_L14N_T2_SRCC_35)
- new net HDMI_D2+: U501.F1 (IO_L18P_T2_35)
- new net HDMI_D2-: U501.E1 (IO_L18N_T2_35)
- new net HDMI_SCL: U501.D3 (IO_L12N_T1_MRCC_35)
- new net HDMI_SDA: U501.E6 (IO_L5P_T0_AD13P_35)
- new net HDMI_~{HPD}: U501.F3 (IO_L13N_T2_MRCC_35)
- new net MCU_~{IRQ}: U501.J3 (IO_L22P_T3_35)
- new net SPI2_CLK: U501.F4 (IO_L13P_T2_MRCC_35)
- new net SPI2_D2: U501.G2 (IO_L15N_T2_DQS_35)
- new net SPI2_D3: U501.H1 (IO_L17P_T2_35)
- new net SPI2_PICO/D0: U501.H2 (IO_L15P_T2_DQS_35)
- new net SPI2_POCI/D1: U501.G1 (IO_L17N_T2_35)
- new net VIBRATE_EN: U501.E7 (IO_L6P_T0_35)
- no-connect marks 0 -> 2
Other:
- note removed: "Bulk decoupling capacitor shared between 4x IO banks sharing same VCCO (3.3V)"
