File: pcb/handheld/gb_cart.kicad_sch (KiCad schematic)
At the start: 23 parts, among them J1301 Cartridge_Slot, U1301 74LVCH16T245, U1302 74LVCH16T245, U20 74LVC1T45, U21 74LVC1T45

Commit message: Rev A of PCB
Parts:
- removed R19: 27R, Resistor_SMD:R_0603_1608Metric_Pad0.98x0.95mm_HandSolder, symbol Device:R_Small
- removed R23 (x2): 47R, Resistor_SMD:R_0402_1005Metric, symbol Device:R_Small
- removed R7: 18k, Resistor_SMD:R_0402_1005Metric, symbol Device:R_Small
- added R1709 (x3): 49R9, Resistor_SMD:R_0402_1005Metric, symbol Device:R_Small
- added R1710: 27K, Resistor_SMD:R_0603_1608Metric, symbol Device:R_Small
- J1901: renamed from J1301; footprint (none) -> Game_Bub:GameBoy_Cartridge_AGS_1x32-1MP_P1.50mm_Socket_Horizontal
- U1901: renamed from U20; LCSC C168855 -> C5162250
- U1903: renamed from U21; LCSC C168855 -> C5162250
- renumbered U1301 to U1902, U1302 to U1904
Connections:
- net Cart_~{CS1}: now also R1709.1
- net Cart_~{CS2}: now also R1709.2
- net Cart_~{WR}: now also R1709.2
- net VGB: now also R1710.1
- net Cart_~{CS1}_d: now reaches J1901.5 (~{CS1}/~{CS})
- net Cart_~{CS1}_d: now also R1709.2
- net Cart_~{WR}_d: now reaches J1901.3 (~{WR})
- net Cart_~{WR}_d: now also R1709.1
- net Cart_~{CS2}_d: now reaches J1901.30 (~{CS2}/~{RES})
- net Cart_~{CS2}_d: now also R1709.1, R1710.2
- net GB_~{OE} renamed GB_Cart_~{OE}
Other:
- moved on the sheet: C1, J1901, R25, U1901, U1903
