File: pcb/handheld/gb_interfaces.kicad_sch (KiCad schematic)
At the start: 12 parts, among them Q3 AO3400A, SW1301 SW_Cartridge, U302 AP2191W

Commit message: Rev A of PCB
Parts:
- added C1 (x2): 100n, Capacitor_SMD:C_0402_1005Metric, symbol Device:C_Small
- SW1901: renamed from SW1301; footprint (none) -> Game_Bub:JJOV0UL650NONPRBK_SIDE
- TP5: renamed from TP3; value +3V3 -> VGB
- renumbered R401 to R1924, R401 to R1925, R11 to R31
Connections:
- net +3V3_FPGA: no longer U302.5 (IN)
- net +5V: now also C1.2
- net GND: now also C1.1, C1.1
- net SW_Cartridge_s: now reaches R31.1, R31.2, SW1901.1 (A)
- net VGB_3V3_SW_En: now reaches Q3.3 (D), R1925.2, R209.2, U302.4 (EN)
- net VGB_5V_SW_En: now reaches Q3.3 (D), R1924.2, R209.2, U302.4 (EN)
- new net +3V3: C1.2, U302.5 (IN)
Other:
- note added: "DMG/CGB: 100mA *max* draw, typical <40mA AGB: 100mA *max*, typical <30mA"
- moved on the sheet: R31, TP5, U302
