File: pcb/handheld/handheld.kicad_sch (KiCad schematic)
At the start: 0 parts

Commit message: Rev A of PCB
Parts:
- added H101, H102, H103: MountingHole, MountingHole:MountingHole_2.7mm_M2.5, symbol Mechanical:MountingHole
Other:
- removed sheet ESP32
- removed sheet FPGA IO 1
- removed sheet FPGA IO 2
- removed sheet FPGA IO 3
- removed sheet RP2040
- added sheet ESP32-S3 (esp32_s3.kicad_sch)
- added sheet FPGA IO Bank 14 (fpga_io_14.kicad_sch)
- added sheet FPGA IO Bank 15 (fpga_io_15.kicad_sch)
- added sheet FPGA IO Bank 16 (fpga_io_16.kicad_sch)
- added sheet FPGA IO Bank 34 (fpga_io_34.kicad_sch)
- added sheet FPGA IO Bank 35 (fpga_io_35.kicad_sch)
- title: (none) -> Game Bub Handheld
