File: pcb/handheld/lcd.kicad_sch (KiCad schematic)
At the start: 9 parts, among them U601 AP2502, U602 AP2502

Commit message: Rev A of PCB
Parts:
- added JP1201: SolderJumper_3_Bridged12, Jumper:SolderJumper-3_P1.3mm_Bridged12_RoundedPad1.0x1.5mm, symbol Jumper:SolderJumper_3_Bridged12
- J1201: renamed from J601; footprint Connector_FFC-FPC:Hirose_FH12-50S-0.5SH_1x50-1MP_P0.50mm_Horizontal -> Game_Bub:Hirose_FH12S-50S-0.5SH_1x50-1MP_P0.50mm_Horizontal_FLIPPED
- renumbered R11 to R1201, U601 to U1201, U602 to U1202
Connections:
- net +3V3: now also JP1201.1 (A)
- net GND: now also JP1201.3 (B); no longer J1201.37 (D/CX), J1201.8 (IM1)
- net LCD_TE: no longer names the net of J1201.39 (TE)
- net SPI0_CLK renamed SPI2_CLK
- net SPI0_PICO renamed SPI2_PICO/D0
- net SPI0_POCI renamed SPI2_POCI/D1
- new net LCD_D/~{CX}: J1201.37 (D/CX)
- new net LCD_IM1: J1201.8 (IM1), JP1201.2 (C)
- no-connect marks 9 -> 7
Other:
- note added: "IM{2, 1, 0} = {1, 1, 1} -> 4-wire, 8-bit SPI"
