File: pcb/handheld/peripherals.kicad_sch (KiCad schematic)
At the start: 15 parts, among them J7 Vibration_Motor, Q3 AO3400A, U1501 LSM6DS3TR-C, U1502 PCF8563T, Y1501 32.768kHz

Commit message: Rev A of PCB
Parts:
- C1405: renamed from C1501; footprint Capacitor_SMD:C_0402_1005Metric -> Capacitor_SMD:C_0402_1005Metric_Pad0.74x0.62mm_HandSolder
- U1402: renamed from U1502; LCSC (none) -> C7440
- renumbered JP1501 to JP1401, JP1502 to JP1402, R10 to R30, R11 to R31, U1501 to U1401, Y1501 to Y1401
Connections:
- net +3V3: no longer C1.1, C1.1, C1.2, C1405.1, Q3.2 (S), R31.2, U1401.1 (SDO/SA0), U1401.2 (SDX), U1401.3 (SCX), U1401.6 (GND), U1401.7 (GND), U1402.4 (VSS)
- net VIBRATE_EN: now also R30.1; no longer R30.2
- net Vibrate_N: now reaches C1.1, D4.2 (A), J7.1 (Pin_1), Q3.3 (D)
- net RTC_OSCI: now reaches C1405.2, U1402.1 (OSCI), Y1401.1
- net RTC_OSCO: now reaches U1402.2 (OSCO), Y1401.2
- net RTC_INT: now reaches JP1402.1 (A), U1402.3 (~{INT})
- net Vibrate_FET_g: now reaches Q3.1 (G)
- net Vibrate_FET_g: now also R30.2; no longer R30.1
- net IMU_INT: now reaches JP1401.1 (A), U1401.4 (INT1)
- net RP2040_~{IRQ} renamed MCU_~{IRQ}
- new net GND: C1.1, C1.1, C1.2, C1405.1, Q3.2 (S), R31.2, U1401.1 (SDO/SA0), U1401.2 (SDX), U1401.3 (SCX), U1401.6 (GND), U1401.7 (GND), U1402.4 (VSS)
Other:
- moved on the sheet: C1405, J7, JP1401, JP1402, R30, R31, Y1401
