File: pcb/handheld/power_path.kicad_sch (KiCad schematic)
At the start: 30 parts, among them J201 Batt_Conn, Q201 AO3401A, Q202 AO3400A, SW201 BTN_POWER, U202 BQ24073RGT, U203 MAX17048

Commit message: Rev A of PCB
Parts:
- removed R14: 1K2, Resistor_SMD:R_0603_1608Metric_Pad0.98x0.95mm_HandSolder, symbol Device:R_Small
- added Q201: AO3400A, Package_TO_SOT_SMD:SOT-23, symbol Transistor_FET:AO3400A
- added R206: 100K, Resistor_SMD:R_0402_1005Metric, symbol Device:R_Small
- added R214: 1K, Resistor_SMD:R_0402_1005Metric_Pad0.72x0.64mm_HandSolder, symbol Device:R_Small
- added R409 (x2): 0R, Resistor_SMD:R_0603_1608Metric_Pad0.98x0.95mm_HandSolder, symbol Device:R_Small
- J201: footprint (none) -> Connector_JST:JST_PH_S2B-PH-K_1x02_P2.00mm_Horizontal
- R201: renamed from R14; footprint Resistor_SMD:R_0402_1005Metric -> Resistor_SMD:R_0603_1608Metric_Pad0.98x0.95mm_HandSolder; LCSC C25900 -> C25819; now not fitted; now left out of the parts list
- R210: renamed from R208; value 300K -> 470K; footprint Resistor_SMD:R_0402_1005Metric -> Resistor_SMD:R_0603_1608Metric_Pad0.98x0.95mm_HandSolder; LCSC C25774 -> C23178
- SW201: value BTN_POWER -> Power; footprint (none) -> Game_Bub:SW_SPST_SKSC; LCSC (none) -> C115361
- renumbered C7 to C201, C204 to C205, C16 to C206, C202 to C207, D206 to D201, D6 to D202, D6 to D203, D201 to D204, Q201 to Q202, Q202 to Q203, R11 to R202, R14 to R203, R201 to R207, R203 to R208, R10 to R211, TP3 to TP201, TP3 to TP202, TP3 to TP203, U203 to U201
Connections:
- net +3V3: now also R206.1
- net GND: now also SW201.2, Q201.2 (S), R214.1, R409.1; no longer SW201.1, U202.6 (EN1)
- net VSYS_ALWAYS: now also R409.1; no longer U202.5 (EN2)
- net ~{CHG}: now also Q201.1 (G)
- net ~{POWER_SW_a}: now reaches D202.2 (A), D203.1 (K), D204.2 (A), R209.2, R210.2, R211.1
- net PWR_TMR: now reaches R201.1, U202.14 (TMR)
- net Charge_LED_A: now reaches D201.2 (A), R33.2
- net BTN_Power_s: now reaches C207.2, D204.1 (K), R207.2
- net BTN_Power_s: now also SW201.1; no longer SW201.2
- net PWR_ILIM: now reaches R203.1, U202.12 (ILIM)
- net PWR_TS: now reaches R202.1, U202.1 (TS)
- net PWR_SW_nFET_g: now reaches C205.2, Q203.1 (G), R210.1
- net PWR_SW_pFET_g: now reaches C206.2, C207.1, Q202.1 (G), Q203.3 (D), R208.2
- net PWR_ISET: now reaches U202.16 (ISET)
- net PWR_ISET: now also R214.2
- net RP2040_~{IRQ} renamed MCU_~{IRQ}
- net ~{PGOOD} renamed ~{VBUS_PGOOD}
- new net BATT_CHG: Q201.3 (D), R206.2
- new net PWR_EN1: R409.2, U202.6 (EN1)
- new net PWR_EN2: R409.2, U202.5 (EN2)
Other:
- note added: "Clamping diodes Protect MCU GPIO from >3.3V or <0V"
- note added: "EN2 = 1, EN1 = 0 --> IN current set with ILIM resistor R_{ILIM} = 1550 AΩ / I = 1550 / 1.5A R_{ILIM} = 1.1 kΩ R_{ISET} = 890 AΩ / I = 890 / 0.89A R_{ISET} = 1.0 kΩ (battery charge current)"
- note added: "Level shifts and inverts the CHG signal allowing for LED to remain lit"
- note removed: "Clamping diodes Protect RP2040 GPIO from >3.3V or <0V"
- note removed: "EN2 = 1, EN1 = 0 --> IN current set with ILIM resistor R_{ILIM} = 1550 AΩ / I = 1550 / 1.5A R_{ILIM} = 1.1 kΩ R_{ISET} = 890 AΩ / I = 890 / 0.75A R_{ISET} = 1.2 kΩ"
- moved on the sheet: C201, C35, D201, D202, D203, J201, R202, R203, R209, R210, R211, R33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
