File: pcb/handheld/power_regulators.kicad_sch (KiCad schematic)
At the start: 41 parts, among them U301 TLV62585PDRL, U302 AP2191W, U304 TPS61023DRLR, U305 LP5907MFX-3.3, U306 TLV62585PDRL, U307 TLV62585PDRL

Commit message: Rev A of PCB
Parts:
- removed U304: TPS61023DRLR, Package_TO_SOT_SMD:SOT-563, symbol Game_Bub:TPS61023DRLR
- added C1: 100n, Capacitor_SMD:C_0402_1005Metric, symbol Device:C_Small
- added U302: TPS61022RWUR, Game_Bub:VQFN-7_L2.0-W2.0-P0.55-TL_RWU, symbol Game_Bub:TPS61022RWUR
- C1501: now left out of the parts list
- JP301: footprint (none) -> Jumper:SolderJumper-3_P1.3mm_Bridged12_RoundedPad1.0x1.5mm
- TP5: renamed from TP3; value +3V3 -> +1V0
- TP5: renamed from TP3; value +3V3 -> +5V
- TP5: renamed from TP3; value +3V3 -> +1V8
- renumbered C18 to C1401, L304 to L302, L302 to L303, L303 to L304, R307 to R303, R303 to R304, R308 to R305, R304 to R306, R305 to R307, R306 to R308, TP3 to TP1, TP3 to TP5, U306 to U303, U307 to U304, U302 to U305, U305 to U306
Connections:
- net +3V3_FPGA_Enable is gone; now on net +1V8_PG: U306.3 (EN)
- net +3V3: now also R25.1, C1.2
- net +5V: now also U302.3 (VOUT)
- net FPGA_POWER_EN: now also U302.5 (EN)
- net GND: now also C1.1, U302.1 (GND), U302.6 (MODE)
- net VSYS: now also U302.7 (VIN); no longer R25.1
- net Buck_3V3_FB: now reaches C1501.1, R307.2, R308.1, U304.5 (FB)
- net Boost_5V_SW: now reaches L302.2
- net Boost_5V_SW: now also U302.2 (SW)
- net Buck_1V0_SW: now reaches L301.1, U301.2 (SW)
- net Buck_1V8_FB: now reaches C1501.1, R304.2, R306.1, U303.5 (FB)
- net Boost_5V_FB: now reaches C1501.1, R303.2, R305.1
- net Boost_5V_FB: now also U302.4 (FB)
- net Buck_1V8_SW: now reaches L303.1, U303.2 (SW)
- net Buck_1V0_FB: now reaches C1501.1, R301.2, R302.1, U301.5 (FB)
- net Buck_3V3_SW: now reaches L304.1, U304.2 (SW)
- net LDO_+3V3_Out: now reaches JP301.3 (B), U306.5 (OUT)
- net +1V0_FPGA renamed +1V0
Other:
- note added: "Vsys -> +3V3 Enable FPGA enable: -> +1V0_FPGA & +5V0 -> +1V8 (FPGA and DAC) -> +3V3 (FPGA and DAC) PG signals are open-drain, active high"
- note removed: "+3V3_FPGA_Enable"
- note removed: "Always: +3V3 FPGA enable: -> +1V0_FPGA & +5V0 -> +1V8_FPGA (& +1V8_DAC) -> +3V3_FPGA (& +3V3_DAC) PG signals are open-drain, active high"
- moved on the sheet: C1401, C1501, C701, JP301, L301, L303, L304, R301, R302, R303, R304, R305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
